File: aprs-esp32/level_shifters.kicad_sch (KiCad schematic)
At the start: 12 parts, among them Q1 BSS138, Q2 BSS138, Q3 BSS138, Q4 BSS138

Commit message: cambios a la lineas de poder
-Modifique la isla de 4v para que sea mas peque;a
-Cambie el ruteo de varios tracks para hacerlos mas cortos
-modificado la ubicacion de algunas vias para que las lineas de tierra esten mas cercanas a los pads
-capacitores de bypass de ESP estan 1mm mas cerca.
Connections:
- net RADIO_RX_HIGH: now also Q2.3 (D), R6.2; no longer Q1.3 (D), R7.2
- net RADIO_RX_LOW: now also Q2.2 (S), R3.2; no longer Q1.2 (S), R4.2
- net RADIO_TX_HIGH: now also Q1.3 (D), R7.2; no longer Q2.3 (D), R6.2
- net RADIO_TX_LOW: now also Q1.2 (S), R4.2; no longer Q2.2 (S), R3.2
Changed lines of the file:
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@@
     )
   )
-  (global_label "RADIO_TX_HIGH" (shape input) (at 147.32 63.5 0) (fields_autoplaced)
+  (global_label "RADIO_TX_HIGH" (shape input) (at 96.52 63.5 0) (fields_autoplaced)
     (effects (font (size 1.27 1.27)) (justify left))
-    (property "Intersheet References" "${INTERSHEET_REFS}" (id 0) (at 163.945 63.4206 0)
+    (property "Intersheet References" "${INTERSHEET_REFS}" (id 0) (at 113.145 63.4206 0)
       (effects (font (size 1.27 1.27)) (justify left) hide)
     )
   )
-  (global_label "RADIO_TX_LOW" (shape input) (at 134.62 63.5 180) (fields_autoplaced)
+  (global_label "RADIO_TX_LOW" (shape input) (at 83.82 63.5 180) (fields_autoplaced)
     (effects (font (size 1.27 1.27)) (justify right))
-    (property "Intersheet References" "${INTERSHEET_REFS}" (id 0) (at 118.7207 63.4206 0)
+    (property "Intersheet References" "${INTERSHEET_REFS}" (id 0) (at 67.9207 63.4206 0)
       (effects (font (size 1.27 1.27)) (justify right) hide)
     )
@@
     )
   )
-  (global_label "RADIO_RX_HIGH" (shape input) (at 96.52 63.5 0) (fields_autoplaced)
+  (global_label "RADIO_RX_HIGH" (shape input) (at 147.32 63.5 0) (fields_autoplaced)
     (effects (font (size 1.27 1.27)) (justify left))
-    (property "Intersheet References" "${INTERSHEET_REFS}" (id 0) (at 113.4474 63.4206 0)
+    (property "Intersheet References" "${INTERSHEET_REFS}" (id 0) (at 164.2474 63.4206 0)
       (effects (font (size 1.27 1.27)) (justify left) hide)
     )
   )
-  (global_label "RADIO_RX_LOW" (shape input) (at 83.82 63.5 180) (fields_autoplaced)
+  (global_label "RADIO_RX_LOW" (shape input) (at 134.62 63.5 180) (fields_autoplaced)
     (effects (font (size 1.27 1.27)) (justify right))
-    (property "Intersheet References" "${INTERSHEET_REFS}" (id 0) (at 67.6183 63.4206 0)
+    (property "Intersheet References" "${INTERSHEET_REFS}" (id 0) (at 118.4183 63.4206 0)
       (effects (font (size 1.27 1.27)) (justify right) hide)
     )
